File: PCB/V2.00/KitchenLightsController V2.brd (EAGLE design)
At the start: 100 x 90 mm, 104 parts, among them IC1 7805, IC2 LM3526M-L, Q2 FDD8451, Q3 FDD8451, Q4 FDD8451, Q5 FDD8451, U1 PHOTON_WITH_STACKABLE_HEADERS, U2 DS1820SOIC, U3 74AHC1G125, U4 INA219AIDCNRSOIC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

Commit message: Added reverse mount LED for OSH Logo.
Modified USB channel B output to drive NeoPixels rather than using the jumper, as NeoPixels have a 1mA per pixel base current consumption this allows a string or NeoPixels to be switched off to save power, as well as providing current limiting etc. as provided by the USB driver chip.
Parts:
- removed JP37: 5V INTERNAL, SparkFun-Connectors:1X02
- removed JP43: 5V Out (USB B), SparkFun-Connectors:SCREWTERMINAL-3.5MM-2
- added D8: (no value), SparkFun-DiscreteSemi:SMA-DIODE-KIT
- added D9: (no value), SparkFun-LED:LED-1206-BOTTOM
- added R20: 1k, SparkFun-Resistors:0805
Connections:
- new net N$9: D9.A, R20.2
- net 5V: now also R20.1; no longer JP37.1
- net GND: now also D9.C; no longer JP43.2
- net USB_VB: now also D8.A; no longer JP43.1
- net VIN: now also D8.C; no longer JP37.2
Routing:
- net VIN: track 47.0 -> 69.3 mm, vias 0 -> 1
- net 5V: track 245.0 -> 251.7 mm, vias 0 -> 1
- net N$9: track 0.00 -> 3.33 mm
Other:
- board text added: "V2.04"
- board text added: "VIn"
- board text removed: "V2.03"
Changed lines of the file:
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@@
 <text x="7.415" y="21.065" size="1.27" layer="25" font="vector">IoT Low Voltage Lights Controller</text>
 <text x="7.415" y="19.16" size="1.016" layer="25" font="vector">(c) Tinamous.com - S.Harrison - 03 April 2016</text>
-<text x="86.79" y="0.745" size="1.016" layer="25" font="vector">V2.03</text>
+<text x="86.79" y="0.745" size="1.016" layer="25" font="vector">V2.04</text>
 <text x="12.685" y="80.12" size="1.778" layer="25">12V DC</text>
 <text x="23.5275" y="85.5175" size="2.54" layer="25">+</text>
@@
 <text x="40.29" y="77.2625" size="2.54" layer="25">2</text>
 <text x="55.4975" y="77.355" size="2.54" layer="25">3</text>
-<text x="67.96" y="77.99" size="2.54" layer="25">4</text>
+<text x="67.96" y="78.625" size="2.54" layer="25">4</text>
 <text x="6.78" y="70.9125" size="0.8128" layer="25">GND</text>
 <text x="6.78" y="73.4525" size="0.8128" layer="25">3v3</text>
 <text x="6.7775" y="76.0875" size="0.8128" layer="25">SCL</text>
 <text x="6.7775" y="78.6275" size="0.8128" layer="25">SDA</text>
-<text x="76.55" y="80.12" size="2.54" layer="25">+</text>
+<text x="76.8675" y="78.215" size="2.54" layer="25">+</text>
 <text x="89.0125" y="63.9275" size="1.27" layer="25" font="vector" rot="R180">5V</text>
 <text x="7.3025" y="17.78" size="1.016" layer="25" font="vector">Github.com/Tinamous/KitchenLightsController</text>
@@
 </polygon>
 <text x="52.42" y="77.2625" size="2.54" layer="25">+</text>
-<text x="65.12" y="80.4375" size="2.54" layer="25">+</text>
+<text x="65.12" y="78.85" size="2.54" layer="25">+</text>
 <text x="37.18" y="76.945" size="2.54" layer="25">+</text>
 <text x="20.67" y="77.2625" size="2.54" layer="25">+</text>
-<text x="86.6775" y="70.8025" size="1.27" layer="25" font="vector" rot="R180">NeoPixels</text>
+<text x="85.725" y="70.8025" size="1.27" layer="25" font="vector" rot="R180">NeoPixels</text>
 <text x="78.74" y="68.8975" size="0.8128" layer="25" font="vector" rot="R180">5V</text>
 <text x="80.9625" y="68.8975" size="0.8128" layer="25" font="vector" rot="R180">D</text>
@@
 <text x="95.045" y="76.31" size="1.27" layer="25" font="vector" rot="R180">12V</text>
 <text x="32.1" y="74.7225" size="1.778" layer="25">+</text>
+<text x="89.535" y="81.915" size="1.016" layer="25" rot="R90">VIn</text>
 </plain>
 <attributes>
@@
 <attribute name="VALUE" x="75.34" y="88.9975" size="1.27" layer="25" rot="R270"/>
 </element>
-<element name="JP37" library="SparkFun-Connectors" package="1X02" value="5V INTERNAL" x="80.44" y="78.85" smashed="yes" rot="R180">
-<attribute name="NAME" x="84.6437" y="79.2437" size="0.8128" layer="25" ratio="10" rot="R180"/>
-</element>
 <element name="C4" library="SparkFun-Capacitors" package="CPOL-RADIAL-1000UF-25V-KIT" value="1000uf/16V" x="80.5325" y="60.85" smashed="yes" rot="R180">
 <attribute name="PROD_ID" value="CAP-09538" x="80.5325" y="60.85" size="1.778" layer="27" rot="R180" display="off"/>
@@
 <attribute name="NAME" x="70.485" y="43.307" size="0.8128" layer="25"/>
 </element>
-<element name="JP43" library="SparkFun-Connectors" package="SCREWTERMINAL-3.5MM-2" value="5V Out (USB B)" x="83.82" y="40.64" smashed="yes" rot="R180">
-<attribute name="PROD_ID" value="CONN-08399" x="83.82" y="40.64" size="0.8128" layer="27" rot="R180" display="off"/>
-<attribute name="VALUE" x="86.36" y="45.72" size="0.8128" layer="27" rot="R180"/>
-</element>
 <element name="R3" library="SparkFun-Resistors" package="0805" value="10k" x="21.2725" y="5.715" smashed="yes" rot="R270">
 <attribute name="NAME" x="19.558" y="4.8895" size="0.8128" layer="25" rot="R270"/>
@@
 <attribute name="NAME" x="18.2245" y="78.867" size="0.8128" layer="25" rot="R180"/>
 </element>
+<element name="D8" library="SparkFun-DiscreteSemi" package="SMA-DIODE-KIT" value="" x="84.1375" y="42.8625" rot="R90"/>
+<element name="D9" library="SparkFun-LED" package="LED-1206-BOTTOM" value="" x="86.0425" y="53.0225" rot="MR270"/>
+<element name="R20" library="SparkFun-Resistors" package="0805" value="1k" x="89.8525" y="55.245" rot="MR0"/>
 </elements>
 <signals>
@@
 <contactref element="U1" pad="1"/>
 <contactref element="U1" pad="@1"/>
-<contactref element="JP37" pad="1"/>
 <wire x1="39.038" y1="31.86" x2="39.165" y2="31.86" width="1.016" layer="1"/>
 <wire x1="39.165" y1="31.86" x2="39.165" y2="34.4" width="1.6764" layer="1"/>
@@
 <wire x1="39.37" y1="34.4" x2="72.39" y2="34.4" width="1.6764" layer="1"/>
 <wire x1="72.39" y1="34.4" x2="93.98" y2="34.4" width="1.6764" layer="1"/>
-<wire x1="97.2675" y1="34.4" x2="97.2675" y2="64.77" width="1.6764" layer="1"/>
+<wire x1="97.2675" y1="34.4" x2="97.2675" y2="55.88" width="1.6764" layer="1"/>
+<wire x1="97.2675" y1="55.88" x2="97.2675" y2="64.77" width="1.6764" layer="1"/>
 <wire x1="97.2675" y1="64.77" x2="97.2675" y2="70.595" width="1.6764" layer="1"/>
 <wire x1="39.038" y1="31.86" x2="39.038" y2="29.32" width="0.8128" layer="1"/>
@@
 <wire x1="73.3425" y1="45.085" x2="73.29" y2="45.72" width="0.6096" layer="1"/>
 <wire x1="87.63" y1="67.31" x2="87.63" y2="70.595" width="0.3048" layer="1"/>
-<wire x1="85.8375" y1="70.595" x2="87.63" y2="70.595" width="1.6764" layer="1"/>
-<wire x1="87.63" y1="70.595" x2="97.2675" y2="70.595" width="1.6764" layer="1"/>
-<wire x1="85.8375" y1="70.595" x2="85.725" y2="70.8025" width="1.6764" layer="1"/>
-<wire x1="85.725" y1="70.8025" x2="85.725" y2="78.74" width="1.6764" layer="1"/>
-<wire x1="85.725" y1="78.74" x2="81.5975" y2="78.74" width="1.6764" layer="1"/>
-<wire x1="81.5975" y1="78.74" x2="80.44" y2="78.85" width="1.6764" layer="1"/>
+<wire x1="87.63" y1="70.595" x2="97.2675" y2="70.595" width="0.4064" layer="1"/>
+<contactref element="R20" pad="1"/>
+<wire x1="90.7525" y1="55.245" x2="97.2675" y2="55.245" width="0.6096" layer="16"/>
+<wire x1="97.2675" y1="55.245" x2="97.2675" y2="55.88" width="0.6096" layer="16"/>
+<via x="97.2675" y="55.88" extent="1-16" drill="0.6"/>
+<wire x1="97.2675" y1="55.88" x2="97.2675" y2="70.595" width="0.6096" layer="1"/>
 </signal>
 <signal name="12V">
@@
 <contactref element="IC2" pad="6"/>
 <wire x1="74.99" y1="40.005" x2="76.5175" y2="40.005" width="0.3048" layer="1"/>
-<contactref element="JP43" pad="2"/>
 <via x="64.135" y="37.465" extent="1-16" drill="0.6" shape="square"/>
 <via x="40.64" y="23.495" extent="1-16" drill="0.6" shape="square"/>
@@
 <via x="60.325" y="75.565" extent="1-16" drill="0.6" shape="square"/>
 <via x="60.325" y="76.835" extent="1-16" drill="0.6" shape="square"/>
+<contactref element="D9" pad="C"/>
+<wire x1="71.49" y1="45.72" x2="74.99" y2="40.005" width="0" layer="19" extent="1-1"/>
 </signal>
 <signal name="VBAT">
@@
 <contactref element="JP35" pad="3"/>
 <contactref element="JP36" pad="1"/>
-<contactref element="JP37" pad="2"/>
-<wire x1="79.0575" y1="86.36" x2="77.9" y2="85.2" width="1.6764" layer="1"/>
-<wire x1="77.9" y1="85.2" x2="77.9" y2="78.85" width="1.6764" layer="1"/>
 <contactref element="C4" pad="+"/>
 <contactref element="R10" pad="2"/>
@@
 <wire x1="80.01" y1="88.9" x2="80.01" y2="87.31" width="0.3048" layer="1"/>
 <wire x1="80.01" y1="87.31" x2="79.0575" y2="86.36" width="0.3048" layer="1"/>
-<wire x1="77.9" y1="78.85" x2="77.9" y2="74.2775" width="1.6764" layer="1"/>
 <wire x1="77.9" y1="74.2775" x2="77.9925" y2="74.185" width="1.016" layer="1"/>
 <wire x1="77.9925" y1="74.185" x2="77.9925" y2="60.89" width="1.6764" layer="1"/>
 <wire x1="77.9925" y1="60.89" x2="78.0325" y2="60.85" width="1.016" layer="1"/>
+<contactref element="D8" pad="C"/>
+<wire x1="79.0575" y1="86.36" x2="77.9925" y2="86.36" width="1.778" layer="1"/>
+<wire x1="77.9925" y1="86.36" x2="77.9925" y2="74.185" width="1.778" layer="1"/>
+<via x="78.105" y="46.99" extent="1-16" drill="0.6"/>
+<wire x1="78.105" y1="46.99" x2="78.0325" y2="48.26" width="1.27" layer="16"/>
+<wire x1="78.0325" y1="48.26" x2="78.0325" y2="60.85" width="1.27" layer="16"/>
+<wire x1="78.105" y1="46.99" x2="84.1375" y2="46.99" width="1.27" layer="1"/>
+<wire x1="84.1375" y1="46.99" x2="84.1375" y2="45.2625" width="1.27" layer="1"/>
 </signal>
 <signal name="D3">
@@
 <signal name="USB_VB">
 <contactref element="IC2" pad="5"/>
-<contactref element="JP43" pad="1"/>
 <wire x1="74.99" y1="38.735" x2="76.5175" y2="38.735" width="0.6096" layer="1"/>
 <wire x1="76.5175" y1="38.735" x2="83.82" y2="38.735" width="1.27" layer="1"/>
-<wire x1="83.82" y1="38.735" x2="83.82" y2="40.64" width="1.27" layer="1"/>
+<contactref element="D8" pad="A"/>
+<wire x1="84.1375" y1="40.4625" x2="83.82" y2="40.4625" width="1.27" layer="1"/>
+<wire x1="83.82" y1="40.4625" x2="83.82" y2="38.735" width="1.27" layer="1"/>
 </signal>
 <signal name="USB_VENABLE_A">
@@
 <wire x1="16.1925" y1="6.615" x2="16.178" y2="9" width="0.6096" layer="1"/>
 </signal>
+<signal name="N$9">
+<contactref element="R20" pad="2"/>
+<contactref element="D9" pad="A"/>
+<wire x1="86.0425" y1="54.8225" x2="88.9525" y2="54.8225" width="0.6096" layer="16"/>
+<wire x1="88.9525" y1="54.8225" x2="88.9525" y2="55.245" width="0.6096" layer="16"/>
+</signal>
 </signals>
