File: PCB/V2.00/KitchenLightsController V2.sch (EAGLE design)
At the start: 116 parts, among them IC1 788TV, Q2 FDD8451, Q3 FDD8451, Q4 FDD8451, Q5 FDD8451, Q6 200mA/50V, U1 PHOTON_WITH_STACKABLE_HEADERS, U2 DS1820SOIC, U3 ACS712

Commit message: Updated with minor tweaks and some additional component values specified from build of the v2.00 board.
Parts:
- added JP41: (no value), SparkFun-Connectors:M04PTH
- C1, C2: value (none) -> 10uF 25V
- C3: value (none) -> 1uF
- C4: value (none) -> 220uF 16V
- D8: value (none) -> 1N4148W
- IC1: value 788TV -> 7805
- JP49: value Button -> Temperature
- Q6: value 200mA/50V -> BSS138
- R2: value 600R -> 330R
- R3: value 10R -> 4k7
- R4: value 10R -> DNP
Connections:
- net GND: now also JP41.1, JP41.2, JP41.3, JP41.4
Other:
- note added: "1 Wire DB18B20+ Temperature Sensors"
- note added: "1.01"
- note added: "12V DC Input"
- note added: "5V PSU"
- note added: "ALT when used with Particle Photon Battery Shield"
- note added: "Add heatsink when driving NeoPixels"
- note added: "Alternativly VIN may be supplied through screw terminal for higher current"
- note added: "Breakout"
- note added: "Button with LED."
- note added: "CPU / Sensors"
- note added: "Can also be used as D0/D1"
- note added: "Check polarity of lights before fitting."
- note added: "Connect to use internal 5V."
- note added: "Current sensor for 12V Only. Does not include VIN for 5V NeoPixel option."
- note added: "DC input and current monitor."
- note added: "Ext. 5V Supply for NeoPixels"
- note added: "External I2C sensors"
- note added: "External Sensor(s)"
- note added: "External light sensor"
- note added: "Lighting"
- note added: "Max 500mA on internal power. Each R|G|B LED = 18mA. R+G+B = 54mA (@100%) * Max 10 White 100% LEDs. * Max 30 R|G|B @100%"
- note added: "Max fuse 5A"
- note added: "Monitor +5V (Photon VIn) Level. Tell if 3.7 LiPol or 5V"
- note added: "NeoPixel Supply."
- note added: "NeoPixels use VIN line. Connect internal 5V to VIN to power from internal, otherwise provide external 5V"
- note added: "Neopixel Driver"
- note added: "On-board SOIC-8 sensor to monitor board temp."
- note added: "Option: If using Particle Photon Battery Shield do not fit IC1. 5V rail comes from Photon VIn pin (3v7 - 5v range). Option: Replace IC1 with connector and use alternative 5V supply or LiPol battery."
- note added: "Photon"
- note added: "Power"
- note added: "Used by Battery Shield. If used externally add 4k7 pull-ups"
- note added: "Uses VIN to drive NeoPixels which may be connected to 5V rail."
- note added: "When running on internal and Photon Battery Shield VIN is Max 3v7 on Battery, 5V on 12V supply"
- note removed: "1.00"
- note removed: "7805"
- note removed: "Connect to use internal 5V regulator."
- note removed: "Monitor VIn Level. Tell if 3.7 LiPol or 5V"
- note removed: "Polarity may be the othere way around on your lights. Check before fitting."
- moved on the sheet: C1, C2, C3, C4, C5, C6, C7, D1, D2, D3, D4, D5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

Commit message: Corrected Gnd/+5V labels on NeoPixel connector which were the wrong way around.
Moved Via from area under Photon as it messed with the text.
Parts:
- removed D8: 1N4148W, SparkFun-DiscreteSemi:DIODESOD123
- removed JP204, JP205, JP206, JP304, JP305, JP306: (no value), SparkFun-Connectors:M02POLAR
- removed JP26, JP31, JP38, JP39, JP4, JP40: (no value), SparkFun-Connectors:M08NO_SILK_FEMALE_PTH
- removed JP29: (no value), SparkFun-Connectors:M05PTH
- removed JP3, JP5, JP7, JP8, JP9: (no value), SparkFun-Connectors:M10NO_SILK_PTH_FEMALE
- removed JP6: (no value), SparkFun-Connectors:M15
- removed Q6: BSS138, SparkFun-DiscreteSemi:MOSFET-NCHANNELBSS138
- added IC2: LM3526M-L, SH-linear:LM3526M-L
- added JP402, JP403: (no value), SparkFun-Connectors:M02POLAR
- added JP42: (no value), SparkFun-Connectors:M15
- added JP43: 5V Out (USB B), SparkFun-Connectors:M023.5MM
- added R19: 4k7, SparkFun-Resistors:RESISTOR0805-RES
- added U4: INA219AIDCNRSOIC, INA219AIDCNR:INA219AIDCNRSOIC
- added X2: PN87520-S, con-berg:PN87520-S
- C1: value 10uF 25V -> 330nF 50V; FARNELL (none) -> 1902922
- C2: value 10uF 25V -> 1uF; device SparkFun-Capacitors:10UF-25V-20%(PTH) -> SparkFun-Capacitors:1UF-25V-10%(0805)"
- C3: value 1uF -> 0.1uF
- C4: value 220uF 16V -> 1000uf/16V; device SparkFun-Capacitors:10UF-25V-20%(PTH) -> SparkFun-Capacitors:1000UF-25V(PTH)KIT; FARNELL (none) -> 9693610
- C6: value 1nF -> 10uF
- C7: value 0.1uF -> 1uF
- F1: FARNELL (none) -> 1453528
- JP1: FARNELL (none) -> 2008197; PLUG (none) -> 2008161
- JP32: device SparkFun-Connectors:M20 -> SparkFun-Connectors:M191X19
- JP34, JP35, JP47, JP48, JP49: FARNELL (none) -> 9731156
- JP36: value LED 5V -> LED Ext. 5V
- R14: value 2k -> 0.1; device SparkFun-Resistors:RESISTOR0805-RES -> SparkFun-Resistors:0.001OHM-3W-1%(2512)3W/1%; FARNELL (none) -> 1435947
- R16: value 10k -> 4k7
- R3: value 4k7 -> 10k
- R4: value DNP -> 10k
- U3: value ACS712 -> 74AHC1G125; device SparkFun-AnalogIC:ACS712 -> SparkFun-DigitalIC:74AHC1G125
Connections:
- net N$31 renamed CHANNEL_4_SWITCHED
- removed net CURRENT_SENSOR: C7.2, D8.C, U1.WKP
- removed net CURRENT_SENSOR_PRE: D8.A, R14.1, R16.1
- removed net D2: U1.D2
- removed net D4: U1.D4
- removed net N$13: Q6.D, R2.1, R3.1
- removed net N$15: C6.1, U3.FILT
- removed net N$28: D2.C, JP301.1, JP302.1, JP303.1, JP304.1, JP305.1, JP306.1, Q3.D
- removed net N$30: D3.C, JP401.1, Q4.D
- removed net N$9: D1.C, JP201.1, JP202.1, JP203.1, JP204.1, JP205.1, JP206.1, Q2.D
- new net CHANNEL_1_SWITCHED: D1.C, JP201.1, JP202.1, JP203.1, Q2.D
- new net CHANNEL_2_SWITCHED: D2.C, JP301.1, JP302.1, JP303.1, Q3.D
- new net CHANNEL_3_SWITCHED: D3.C, JP401.1, JP402.1, JP403.1, Q4.D
- new net USB_VA: IC2.OUTA, X2.1
- new net USB_VB: IC2.OUTB, JP43.1
- new net USB_VENABLE_A: IC2.!ENA, R3.1, U1.D4
- new net USB_VENABLE_B: IC2.!ENB, R4.1, U1.D2
- new net WKP: U1.WKP
- net 12V: now also JP402.2, JP403.2, R14.2, U4.VIN-; no longer JP204.2, JP205.2, JP206.2, JP304.2, JP305.2, JP306.2, R5.2, U3.IP-@3, U3.IP-@4
- net 3.3V: now also C5.2, C6.2, R16.1, R19.1, R3.2, U4.VS; no longer JP32.20, Q6.G
- net 5V: now also C2.2, C7.2, IC2.IN, JP42.1, JP42.10, JP42.11, JP42.12, JP42.13, JP42.14, JP42.15, JP42.2, JP42.3, JP42.4, JP42.5, JP42.6, JP42.7, JP42.8, JP42.9; no longer C2.+, C5.2, JP29.1, JP29.2, JP29.3, JP29.4, JP29.5, U3.VCC
- net GND: now also C2.1, C6.1, IC2.GND, JP43.2, U3./OE, U4.A0, U4.A1, U4.GND, X2.4, X2.S1, X2.S2; no longer C2.-, C6.2, JP6.1, JP6.10, JP6.11, JP6.12, JP6.13, JP6.14, JP6.15, JP6.2, JP6.3, JP6.4, JP6.5, JP6.6, JP6.7, JP6.8, JP6.9, R16.2
- net N$5: now also R14.1, R5.2, U4.VIN+; no longer U3.IP+@1, U3.IP+@2
- net N$6: now also R2.1, U3.Y; no longer R14.2, U3.VOUT
- net NEOPIXELS: now also U3.A; no longer Q6.S, R4.1
- net SCL: now also R16.2, U4.SCL
- net SDA: now also R19.2, U4.SDA
- net VIN: now also U3.VCC; no longer R3.2
Other:
- note added: "2.02"
- note added: "5V Control. USB A Socket and 2 pin header source for 5V."
- note added: "ALERT when used with Particle Photon Battery Shield"
- note added: "I2C Pullups"
- note removed: "0-5v -> 0-3v3 divider"
- note removed: "1.01"
- note removed: "ALT when used with Particle Photon Battery Shield"
- moved on the sheet: C1, C3, C5, C6, C7, D1, D2, D3, D4, D5, D6, D7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

Commit message: Added reverse mount LED for OSH Logo.
Modified USB channel B output to drive NeoPixels rather than using the jumper, as NeoPixels have a 1mA per pixel base current consumption this allows a string or NeoPixels to be switched off to save power, as well as providing current limiting etc. as provided by the USB driver chip.
Parts:
- removed JP37: 5V INTERNAL, SparkFun-Connectors:M02PTH
- removed JP43: 5V Out (USB B), SparkFun-Connectors:M023.5MM
- added D8: (no value), SparkFun-DiscreteSemi:DIODESMA-KIT
- added D9: (no value), SparkFun-LED:LED1206-BOTTOM
- added R20: 1k, SparkFun-Resistors:RESISTOR0805-RES
Connections:
- new net N$9: D9.A, R20.2
- net 5V: now also R20.1; no longer JP37.1
- net GND: now also D9.C; no longer JP43.2
- net USB_VB: now also D8.A; no longer JP43.1
- net VIN: now also D8.C; no longer JP37.2
Other:
- note added: "2.04"
- note added: "ALT when used with Particle Photon Battery Shield"
- note added: "Enable USB_VB to use internal 5V supply to power NeoPixels."
- note added: "NeoPixels use VIN line. Connect internal 5V to VIN using USB switch Channel B to power from internal 5V regulator. Otherwise provide external 5V"
- note removed: "2.02"
- note removed: "ALERT when used with Particle Photon Battery Shield"
- note removed: "Connect to use internal 5V."
- note removed: "NeoPixels use VIN line. Connect internal 5V to VIN to power from internal, otherwise provide external 5V"
